File: SolarCellZ_v1.sch (KiCad schematic (older format))
At the start: 28 parts, among them IC1 TSL2561, J1 XF2M-1015-1A, Q1 IRLML2803, U1 NDS8434

Commit message: fixed schematic / pcb mismatch
Parts:
- removed C1: 0.1uF, Capacitor_SMD:C_0402_1005Metric, symbol SolarCellZ_v1-rescue:0.1UF-0603-25V-(+80_-20%)-misc-circuits-cache-misc-circuit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
- removed R1, R2, R6: 0, Resistor_SMD:R_0402_1005Metric, symbol SolarCellZ_v1-rescue:0OHM-0603-1_10W-5%-misc-circuits-cache-misc-circuits-rescue
- added C1: 1.0uF, Capacitor_SMD:C_0402_1005Metric, symbol SolarCellX_v3-rescue:1.0UF-0603-16V-10%-misc-circuits-cache-misc-circuits-rescue
- added C10, C13, C2, C9: 0.1uF, Capacitor_SMD:C_0402_1005Metric, symbol SolarCellX_v3-rescue:0.1UF-0603-25V-(+80_-20%)-misc-circuits-cache-misc-circuit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
- added C11, C12, C14, C6: 100uF, Capacitor_SMD:C_0603_1608Metric, symbol SolarCellX_v3-rescue:0.1UF-0603-25V-(+80_-20%)-misc-circuits-cache-misc-circuit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
- added C3, C8: 4.7uF, Capacitor_SMD:C_0402_1005Metric, symbol SolarCellX_v3-rescue:4.7UF0603-misc-circuits-cache-misc-circuits-rescue
- added C4: 10nF, Capacitor_SMD:C_0402_1005Metric, symbol SolarCellX_v3-rescue:10NF-0603-50V-10%-misc-circuits-cache-misc-circuits-rescue
- added C5: 0.1uF, Capacitor_SMD:C_0402_1005Metric, symbol SolarCellZ_v1-rescue:0.1UF-0603-25V-(+80_-20%)-misc-circuits-cache-misc-circuit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
- added C7: 22uF, Capacitor_SMD:C_0402_1005Metric, symbol SolarCellX_v3-rescue:22UF-0805-6.3V-20%-misc-circuits-cache-misc-circuits-rescue
- added D1: SDM20U40-7, misc-circuits:SOD523, symbol SolarCellX_v3-rescue:DIODE-SOD523-misc-circuits-cache-misc-circuits-rescue
- added D2: MSS1P4-M3_89A, misc-circuits:MICROSMP, symbol SolarCellX_v3-rescue:MSS1P4-M3_89A-symbols
- added L1: 22uH-LPS4018-223MR, misc-circuits:LPS4018, symbol SolarCellX_v3-rescue:COILCRAFT-LPS4018-misc-circuits-cache-misc-circuits-rescue
- added L2: 10uH-LPS4018-103MR, misc-circuits:LPS4018, symbol SolarCellX_v3-rescue:COILCRAFT-LPS4018-misc-circuits-cache-misc-circuits-rescue
- added R1, R14, R15, R16, R17, R18, R2, R20, R21, R22: 0, Resistor_SMD:R_0402_1005Metric, symbol SolarCellX_v3-rescue:0OHM-0603-1_10W-5%-misc-circuits-cache-misc-circuits-rescue
- added R10, R8: 8.25M, Resistor_SMD:R_0402_1005Metric, symbol SolarCellX_v3-rescue:1MOHM-0603-1_4W-5%-misc-circuits-cache-misc-circuits-rescue
- added R11: 4.75M, Resistor_SMD:R_0402_1005Metric, symbol SolarCellX_v3-rescue:1MOHM-0603-1_4W-5%-misc-circuits-cache-misc-circuits-rescue
- added R12, R13: 0, Resistor_SMD:R_0402_1005Metric, symbol SolarCellZ_v1-rescue:0OHM-0603-1_10W-5%-misc-circuits-cache-misc-circuits-rescue
- added R5: 7.32M, Resistor_SMD:R_0402_1005Metric, symbol SolarCellX_v3-rescue:1MOHM-0603-1_4W-5%-misc-circuits-cache-misc-circuits-rescue
- added R6: 5.62M, Resistor_SMD:R_0402_1005Metric, symbol SolarCellX_v3-rescue:1MOHM-0603-1_4W-5%-misc-circuits-cache-misc-circuits-rescue
- added R7: 374K, Resistor_SMD:R_0402_1005Metric, symbol SolarCellX_v3-rescue:1MOHM-0603-1_4W-5%-misc-circuits-cache-misc-circuits-rescue
- added R9: 4.53M, Resistor_SMD:R_0402_1005Metric, symbol SolarCellX_v3-rescue:1MOHM-0603-1_4W-5%-misc-circuits-cache-misc-circuits-rescue
- added U2: Value, misc-circuits:QFN50P350X350X100-21N-D, symbol SolarCellX_v3-rescue:BQ25570RGRR-misc-circuits-cache-misc-circuits-rescue
- D3: renamed from D1; footprint custom-footprints:MICROSMP -> misc-circuits:MICROSMP
- renumbered D2 to D4, D3 to D5, R5 to R19
Connections:
- net labels added: VBAT, VBAT_OK, VOUT_EN
- wire segments 63 -> 175
Other:
- note added: "80% MPPT"
- note added: "BQ25570RGRR"
- note added: "COIL+"
- note added: "COIL-"
- note added: "Clockwise\n(while facing layer 1)"
- note added: "DNI"
- note added: "Energy Harvesting IC"
- note added: "External energy storage\nInput/Output"
- note added: "External\nPower Source\nInput\n(Solar)"
- note added: "Imin=280uA"
- note added: "MPPT Set Resistors"
- note added: "Sets of resistor dividers should = 13MOhm"
- note added: "VBAT_OK\nON: 3.51V\nOFF: 3.42V"
- note added: "VBAT_OV\n4.2V"
- note added: "VOUT=1.21V*((ROUT2+ROUT1)/ROUT1)"
- note added: "VOUT\n3.31"
- note added: "ZENER"
- moved on the sheet: D3, D4, D5, JP1, Q1, R19, R3, R4, SC1, SC2, SC3, SC4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
